File: 01_Hardware/ElectronicsV3/ElectronicsV3.kicad_sch (KiCad schematic)
At the start: 32 parts, among them J1 Filter_CH1_1out, J2 Filter_CH1_2out, J3 Filter_CH1_2in, J4 Filter_CH1_1in, M1 NEMA17_Stepper, U1 ADS1115, U2 EL817, U3 LM1117T-3.3, U4 EL817

Commit message: V3.1
Parts:
- C1: value 330uF -> 47uF
- C2: value 330uF -> 10uF
- R1, RV1: value R10k -> R5k
Connections:
- net GNDA: now also R1.1
- net GNDPWR: no longer R1.1
- net at R11.1: now also MCU1.13 (ADC2_CH2); no longer MCU1.4 (ADC1_CH3)
- net at MCU1.2 (ADC1_CH1): no longer R9.1
- new net: MCU1.4 (ADC1_CH3), R9.1
Other:
- note added: "1.4"
- note added: "2025-10-20"
- note removed: "1.3"
- note removed: "2025-10-07"
Changed lines of the file:
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@@
 		)
 	)
-	(text "1.3"
+	(text "1.4"
 		(exclude_from_sim no)
 		(at 268.478 192.786 0)
@@
 		)
 	)
-	(text "2025-10-07"
+	(text "2025-10-20"
 		(exclude_from_sim no)
 		(at 206.248 192.532 0)
@@
 		)
 	)
-	(text_box "Replace both gain potmeters with constant resistor of R98.8 for a 501 gain"
+	(text_box "Replace both gain potmeters with constant resistor of R91 for a 544 gain"
 		(exclude_from_sim no)
 		(at 201.93 132.08 0)
@@
 	(wire
 		(pts
+			(xy 81.28 63.5) (xy 119.38 63.5)
+		)
+		(stroke
+			(width 0)
+			(type default)
+		)
+	)
+	(wire
+		(pts
+			(xy 58.42 58.42) (xy 119.38 58.42)
+		)
+		(stroke
+			(width 0)
+			(type default)
+		)
+	)
+	(wire
+		(pts
 			(xy 59.69 128.27) (xy 59.69 130.81)
 		)
@@
 	(wire
 		(pts
-			(xy 168.91 97.79) (xy 179.07 97.79)
+			(xy 81.28 64.77) (xy 81.28 63.5)
 		)
 		(stroke
@@
 	(wire
 		(pts
-			(xy 157.48 27.94) (xy 162.56 27.94)
+			(xy 168.91 97.79) (xy 179.07 97.79)
 		)
 		(stroke
@@
 	(wire
 		(pts
-			(xy 171.45 121.92) (xy 170.18 121.92)
+			(xy 157.48 27.94) (xy 162.56 27.94)
 		)
 		(stroke
@@
 	(wire
 		(pts
-			(xy 179.07 127) (xy 179.07 140.97)
+			(xy 171.45 121.92) (xy 170.18 121.92)
 		)
 		(stroke
@@
 	(wire
 		(pts
-			(xy 58.42 55.88) (xy 119.38 55.88)
+			(xy 179.07 127) (xy 179.07 140.97)
 		)
 		(stroke
@@
 	(wire
 		(pts
-			(xy 58.42 64.77) (xy 58.42 55.88)
+			(xy 53.34 100.33) (xy 54.61 100.33)
 		)
 		(stroke
@@
 	(wire
 		(pts
-			(xy 53.34 100.33) (xy 54.61 100.33)
+			(xy 54.61 100.33) (xy 54.61 107.95)
 		)
 		(stroke
@@
 	(wire
 		(pts
-			(xy 54.61 100.33) (xy 54.61 107.95)
+			(xy 146.05 27.94) (xy 149.86 27.94)
 		)
 		(stroke
@@
 	(wire
 		(pts
-			(xy 146.05 27.94) (xy 149.86 27.94)
+			(xy 86.36 71.12) (xy 86.36 73.66)
 		)
 		(stroke
@@
 	(wire
 		(pts
-			(xy 86.36 71.12) (xy 86.36 73.66)
+			(xy 39.37 88.9) (xy 43.18 88.9)
 		)
 		(stroke
@@
 	(wire
 		(pts
-			(xy 39.37 88.9) (xy 43.18 88.9)
+			(xy 218.44 106.68) (xy 231.14 106.68)
 		)
 		(stroke
@@
 	(wire
 		(pts
-			(xy 218.44 106.68) (xy 231.14 106.68)
+			(xy 58.42 64.77) (xy 58.42 58.42)
 		)
 		(stroke
@@
 	(wire
 		(pts
-			(xy 81.28 58.42) (xy 81.28 64.77)
-		)
-		(stroke
-			(width 0)
-			(type default)
-		)
-	)
-	(wire
-		(pts
 			(xy 170.18 121.92) (xy 170.18 125.73)
 		)
@@
 	(wire
 		(pts
-			(xy 119.38 58.42) (xy 81.28 58.42)
-		)
-		(stroke
-			(width 0)
-			(type default)
-		)
-	)
-	(wire
-		(pts
 			(xy 191.77 114.3) (xy 189.23 114.3)
 		)
@@
 			)
 		)
-		(property "Value" "330uF"
-			(at 169.164 75.946 90)
+		(property "Value" "10uF"
+			(at 161.544 76.454 90)
 			(effects
 				(font
@@
 			)
 		)
-		(property "Value" "330uF"
+		(property "Value" "47uF"
 			(at 170.18 99.06 90)
 			(effects
@@
 			)
 		)
-		(property "Value" "R10k"
+		(property "Value" "R5k"
 			(at 153.67 19.558 90)
 			(effects
@@
 			)
 		)
-		(property "Value" "R10k"
+		(property "Value" "R5k"
 			(at 153.67 29.972 90)
 			(effects
@@
 	(symbol
 		(lib_id "power:GNDA")
+		(at 162.56 21.59 90)
+		(unit 1)
+		(exclude_from_sim no)
+		(in_bom yes)
+		(on_board yes)
+		(dnp no)
+		(fields_autoplaced yes)
+		(property "Reference" "#PWR019"
+			(at 168.91 21.59 0)
+			(effects
+				(font
+					(size 1.27 1.27)
+				)
+				(hide yes)
+			)
+		)
+		(property "Value" "GNDA"
+			(at 166.37 21.5899 90)
+			(effects
+				(font
+					(size 1.27 1.27)
+				)
+				(justify right)
+			)
+		)
+		(property "Footprint" ""
+			(at 162.56 21.59 0)
+			(effects
+				(font
+					(size 1.27 1.27)
+				)
+				(hide yes)
+			)
+		)
+		(property "Datasheet" ""
+			(at 162.56 21.59 0)
+			(effects
+				(font
+					(size 1.27 1.27)
+				)
+				(hide yes)
+			)
+		)
+		(property "Description" "Power symbol creates a global label with name \"GNDA\" , analog ground"
+			(at 162.56 21.59 0)
+			(effects
+				(font
+					(size 1.27 1.27)
+				)
+				(hide yes)
+			)
+		)
+		(pin "1"
+		)
+		(instances
+			(project "ElectronicsV3"
+				(path "/f4854c19-51dc-42b5-a843-faca72143437"
+					(reference "#PWR019")
+					(unit 1)
+				)
+			)
+		)
+	)
+	(symbol
+		(lib_id "power:GNDA")
 		(at 196.85 124.46 270)
 		(unit 1)
@@
 					(unit 1)
 				)
-			)
-		)
-	)
-	(symbol
-		(lib_id "power:GNDREF")
-		(at 162.56 21.59 90)
-		(unit 1)
-		(exclude_from_sim no)
-		(in_bom yes)
-		(on_board yes)
-		(dnp no)
-		(fields_autoplaced yes)
-		(property "Reference" "#PWR01"
-			(at 168.91 21.59 0)
-			(effects
-				(font
-					(size 1.27 1.27)
-				)
-				(hide yes)
-			)
-		)
-		(property "Value" "GNDREF"
-			(at 167.64 21.59 0)
-			(effects
-				(font
-					(size 1.27 1.27)
-				)
-				(hide yes)
-			)
-		)
-		(property "Footprint" ""
-			(at 162.56 21.59 0)
-			(effects
-				(font
-					(size 1.27 1.27)
-				)
-				(hide yes)
-			)
-		)
-		(property "Datasheet" ""
-			(at 162.56 21.59 0)
-			(effects
-				(font
-					(size 1.27 1.27)
-				)
-				(hide yes)
-			)
-		)
-		(property "Description" "Power symbol creates a global label with name \"GNDREF\" , reference supply ground"
-			(at 162.56 21.59 0)
-			(effects
-				(font
-					(size 1.27 1.27)
-				)
-				(hide yes)
-			)
-		)
-		(pin "1"
-		)
-		(instances
-			(project ""
-				(path "/f4854c19-51dc-42b5-a843-faca72143437"
-					(reference "#PWR01")
-					(unit 1)
-				)

Commit message: V3.2
Parts:
- R10, R8: value R200 -> R750
- R11, R9: value R1k -> R36
Connections:
- net GNDA: now also R11.1, R9.1; no longer U2.2, U4.2
- net GNDPWR: now also U2.3, U4.3; no longer R10.1, R8.1
- net at MCU1.13 (ADC2_CH2): no longer R11.1
- net at R11.2: now also U4.2; no longer U4.1
- net at A1.10 (M0), A1.11 (M1), A1.12 (M2)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: now also R10.2, R8.2; no longer U2.4, U4.4
- net at MCU1.2 (ADC1_CH1): now also U2.1
- net at MCU1.4 (ADC1_CH3): now also U4.1; no longer R9.1
- net at R9.2: now also U2.2; no longer U2.1
- new net: A1.15 (STEP), R10.1, U4.4
- new net: A1.16 (DIR), R8.1, U2.4
Other:
- moved on the sheet: R10, R11, R8, R9, V1

Commit message: Version Torque 2026
Parts:
- added D1: LED, symbol Device:LED
- R1, RV1: value R5k -> 5kΩ
- R10, R8: value R750 -> 750Ω
- R11, R9: value R36 -> 36Ω
- V2: value +24V -> +15V
- renumbered R4 to 350Ω, R5 to 350Ω
Connections:
- net at A1.10 (M0), A1.11 (M1), A1.12 (M2)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: now also D1.2 (A)
- net at A1.2 (~{FLT}): now also D1.1 (K)
- net +24V: no longer names the net of A1.8 (VMOT), C5.2, V2.1
Other:
- note added: "2.0"
- note added: "2025-11-27"
- note removed: "1.4"
- note removed: "2025-10-20"
